File: PCB/Project_241/SENS.kicad_sch (KiCad schematic)
At the start: 14 parts, among them J2 Wind_Hall, J5 Rain_Hall, U3 HDC1080, U5 LM393

Commit message: Update pcb and doc folder
Parts:
- removed R7: 150R, symbol Device:R_Small
- removed U5: LM393, symbol Comparator:LM393
- added R12: 10k, symbol Device:R_Small
- added U3: LM393, symbol Comparator:LM393
- R3: value 150R -> 10k
- renumbered U3 to U5
Connections:
- net +5V: now also R3.2, R12.2, U3.4 (V-)
- net GND: now also U3.8 (V+)
- net RAIN_GAUSE: now also R12.1, U3.7
- net WIND_SPEED: now also R3.1, U3.1
- net at R6.1: now also J2.2 (Pin_2), U3.2 (-); no longer R3.2
- net at J5.2 (Pin_2): now also R8.1, U3.6 (-)
- net at RV2.2: now also U3.5 (+)
- net at RV1.2: now also U3.3 (+)
Other:
- moved on the sheet: C11
