File: PCB/Project_241/Project_241.kicad_sch (KiCad schematic)
At the start: 0 parts

Commit message: update gerber
Other:
- sheet LORA ports: added LORA_RESET; removed RESET
- sheet MCU ports: added GPS_RX, GPS_TX, LORA_RESET; removed RESET
- sheet SENS ports: added GPS_RX, GPS_TX; removed none
Changed lines of the file:
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@@
 	(wire
 		(pts
-			(xy 170.18 118.11) (xy 182.88 118.11)
-		)
-		(stroke
-			(width 0)
-			(type default)
-		)
-	)
-	(wire
-		(pts
-			(xy 170.18 115.57) (xy 182.88 115.57)
+			(xy 170.18 123.698) (xy 182.88 123.698)
+		)
+		(stroke
+			(width 0)
+			(type default)
+		)
+	)
+	(wire
+		(pts
+			(xy 170.18 121.158) (xy 182.88 121.158)
+		)
+		(stroke
+			(width 0)
+			(type default)
+		)
+	)
+	(wire
+		(pts
+			(xy 170.18 117.856) (xy 182.88 117.856)
 		)
 		(stroke
@@
 		(pts
 			(xy 170.18 78.74) (xy 182.88 78.74)
+		)
+		(stroke
+			(width 0)
+			(type default)
+		)
+	)
+	(wire
+		(pts
+			(xy 170.18 115.062) (xy 182.88 115.062)
 		)
 		(stroke
@@
 	(sheet
 		(at 182.88 104.14)
-		(size 24.384 17.78)
+		(size 24.384 25.146)
 		(fields_autoplaced yes)
 		(stroke
@@
 		)
 		(property "Sheetfile" "SENS.kicad_sch"
-			(at 182.88 122.5046 0)
+			(at 182.88 129.8706 0)
 			(effects
 				(font
@@
 		)
 		(pin "RAIN_GAUSE" input
-			(at 182.88 115.57 180)
+			(at 182.88 121.158 180)
 			(effects
 				(font
@@
 		)
 		(pin "WIND_SPEED" input
-			(at 182.88 118.11 180)
+			(at 182.88 123.698 180)
+			(effects
+				(font
+					(size 1.27 1.27)
+				)
+				(justify left)
+			)
+		)
+		(pin "GPS_TX" input
+			(at 182.88 115.062 180)
+			(effects
+				(font
+					(size 1.27 1.27)
+				)
+				(justify left)
+			)
+		)
+		(pin "GPS_RX" input
+			(at 182.88 117.856 180)
 			(effects
 				(font
@@
 			)
 		)
-		(pin "RESET" input
-			(at 182.88 76.2 180)
-			(effects
-				(font
-					(size 1.27 1.27)
-				)
-				(justify left)
-			)
-		)
 		(pin "NSS" input
 			(at 182.88 78.74 180)
+			(effects
+				(font
+					(size 1.27 1.27)
+				)
+				(justify left)
+			)
+		)
+		(pin "LORA_RESET" input
+			(at 182.88 76.2 180)
 			(effects
 				(font
@@
 	(sheet
 		(at 119.634 72.39)
-		(size 50.546 51.054)
+		(size 50.546 56.896)
 		(fields_autoplaced yes)
 		(stroke
@@
 		)
 		(property "Sheetfile" "MCU.kicad_sch"
-			(at 119.634 124.0286 0)
+			(at 119.634 129.8706 0)
 			(effects
 				(font
@@
 		)
 		(pin "WIND_SPEED" input
-			(at 170.18 118.11 0)
+			(at 170.18 123.698 0)
 			(effects
 				(font
@@
 		)
 		(pin "RAIN_GAUSE" input
-			(at 170.18 115.57 0)
+			(at 170.18 121.158 0)
 			(effects
 				(font
@@
 			)
 		)
-		(pin "RESET" input
+		(pin "GPS_RX" input
+			(at 170.18 117.856 0)
+			(effects
+				(font
+					(size 1.27 1.27)
+				)
+				(justify right)
+			)
+		)
+		(pin "GPS_TX" input
+			(at 170.18 115.062 0)
+			(effects
+				(font
+					(size 1.27 1.27)
+				)
+				(justify right)
+			)
+		)
+		(pin "LORA_RESET" input
 			(at 170.18 76.2 0)
 			(effects
